File: PSU-NONISOLATED.kicad_pcb (KiCad board)
At the start: 2 copper layers, 81.5 x 20 mm, 21 parts, among them J1 Mains, J2 DC, U1 LNK306D

Commit message: Description and some silkscreen for v2
Other:
- board text added: "NEUTRAL"
Changed lines of the file:
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@@
+    (effects (font (size 1 1) (thickness 0.15)))
+  )
+  (gr_text "NEUTRAL" (at 68.2 63.45) (layer "F.SilkS")
     (effects (font (size 1 1) (thickness 0.15)))
   )
